File: led driver.sch (EAGLE design)
At the start: 12 parts, among them IC1 MEGA8-AI, Q1 BC639, Q2 BC640, Q3 IRF540, U1 MAX485CSA+

Commit message: led driver sch and pcb
Parts:
- Q1: value BC639 -> BCP56
- Q2: value BC640 -> BCP53
Connections:
- removed net N$12: F1.2, LED-1.S
- new net N$13: C1.1, F1.1, LED-1.S
- net +12V: now also F1.2; no longer C1.1, F1.1
- net N$6: no longer R2.1
- net N$7: now also R2.1
Other:
- moved on the sheet: F1
Changed lines of the file:
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@@
 <setting verticaltext="up"/>
 </settings>
-<grid distance="0.1" unitdist="inch" unit="inch" style="lines" multiple="1" display="yes" altdistance="0.01" altunitdist="inch" altunit="inch"/>
+<grid distance="0.1" unitdist="inch" unit="inch" style="lines" multiple="1" display="no" altdistance="0.01" altunitdist="inch" altunit="inch"/>
 <layers>
 <layer number="1" name="Top" color="4" fill="1" visible="no" active="no"/>
@@
 <part name="GND3" library="supply1" deviceset="GND" device=""/>
 <part name="R2" library="resistor" deviceset="R-EU_" device="R1206" value="22"/>
-<part name="Q1" library="transistor-small-signal" deviceset="BC639" device=""/>
-<part name="Q2" library="transistor-small-signal" deviceset="BC640" device=""/>
+<part name="Q1" library="transistor-small-signal" deviceset="BC639" device="" value="BCP56"/>
+<part name="Q2" library="transistor-small-signal" deviceset="BC640" device="" value="BCP53"/>
 <part name="P+3" library="supply1" deviceset="VCC" device=""/>
 <part name="GND4" library="supply1" deviceset="GND" device=""/>
@@
 <instance part="GND5" gate="1" x="147.32" y="111.76"/>
 <instance part="C1" gate="G$1" x="147.32" y="137.16"/>
-<instance part="P+5" gate="1" x="147.32" y="147.32"/>
-<instance part="F1" gate="1" x="162.56" y="142.24"/>
+<instance part="P+5" gate="1" x="147.32" y="160.02"/>
+<instance part="F1" gate="1" x="147.32" y="149.86" rot="R90"/>
 <instance part="LED" gate="-1" x="172.72" y="142.24" smashed="yes">
 <attribute name="NAME" x="175.26" y="141.478" size="1.524" layer="95"/>
@@
 <pinref part="ISP" gate="-1" pin="S"/>
 <wire x1="93.98" y1="66.04" x2="119.38" y2="66.04" width="0.1524" layer="91"/>
-<wire x1="93.98" y1="66.04" x2="93.98" y2="119.38" width="0.1524" layer="91"/>
-<pinref part="R2" gate="G$1" pin="1"/>
-<wire x1="93.98" y1="119.38" x2="96.52" y2="119.38" width="0.1524" layer="91"/>
-<junction x="93.98" y="66.04"/>
 </segment>
 </net>
@@
 <pinref part="ISP" gate="-9" pin="S"/>
 <wire x1="109.22" y1="45.72" x2="119.38" y2="45.72" width="0.1524" layer="91"/>
+<wire x1="109.22" y1="45.72" x2="109.22" y2="96.52" width="0.1524" layer="91"/>
+<pinref part="R2" gate="G$1" pin="1"/>
+<wire x1="109.22" y1="96.52" x2="93.98" y2="96.52" width="0.1524" layer="91"/>
+<wire x1="93.98" y1="96.52" x2="93.98" y2="119.38" width="0.1524" layer="91"/>
+<wire x1="93.98" y1="119.38" x2="96.52" y2="119.38" width="0.1524" layer="91"/>
+<junction x="109.22" y="45.72"/>
 </segment>
 </net>
@@
 </segment>
 </net>
+<net name="N$13" class="0">
+<segment>
+<pinref part="C1" gate="G$1" pin="1"/>
+<pinref part="F1" gate="1" pin="1"/>
+<wire x1="147.32" y1="144.78" x2="147.32" y2="142.24" width="0.1524" layer="91"/>
+<pinref part="LED" gate="-1" pin="S"/>
+<wire x1="147.32" y1="142.24" x2="147.32" y2="139.7" width="0.1524" layer="91"/>
+<wire x1="170.18" y1="142.24" x2="147.32" y2="142.24" width="0.1524" layer="91"/>
+<junction x="147.32" y="142.24"/>
+</segment>
+</net>
 <net name="+12V" class="0">
 <segment>
-<pinref part="C1" gate="G$1" pin="1"/>
 <pinref part="P+5" gate="1" pin="+12V"/>
-<wire x1="147.32" y1="139.7" x2="147.32" y2="142.24" width="0.1524" layer="91"/>
-<pinref part="F1" gate="1" pin="1"/>
-<wire x1="147.32" y1="142.24" x2="147.32" y2="144.78" width="0.1524" layer="91"/>
-<wire x1="147.32" y1="142.24" x2="157.48" y2="142.24" width="0.1524" layer="91"/>
-<junction x="147.32" y="142.24"/>
-</segment>
-</net>
-<net name="N$12" class="0">
-<segment>
 <pinref part="F1" gate="1" pin="2"/>
-<pinref part="LED" gate="-1" pin="S"/>
-<wire x1="167.64" y1="142.24" x2="170.18" y2="142.24" width="0.1524" layer="91"/>
-</segment>
-</net>
+<wire x1="147.32" y1="157.48" x2="147.32" y2="154.94" width="0.1524" layer="91"/>
+</segment>
+</net>

Commit message: led driver corrected, led driver test code
Connections:
- net N$6: now also R2.1
- net N$7: no longer R2.1
Changed lines of the file:
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@@
 <pinref part="ISP" gate="-1" pin="S"/>
 <wire x1="93.98" y1="66.04" x2="119.38" y2="66.04" width="0.1524" layer="91"/>
+<pinref part="R2" gate="G$1" pin="1"/>
+<wire x1="93.98" y1="119.38" x2="96.52" y2="119.38" width="0.1524" layer="91"/>
+<wire x1="93.98" y1="66.04" x2="93.98" y2="119.38" width="0.1524" layer="91"/>
+<junction x="93.98" y="66.04"/>
 </segment>
 </net>
@@
 <pinref part="ISP" gate="-9" pin="S"/>
 <wire x1="109.22" y1="45.72" x2="119.38" y2="45.72" width="0.1524" layer="91"/>
-<wire x1="109.22" y1="45.72" x2="109.22" y2="96.52" width="0.1524" layer="91"/>
-<pinref part="R2" gate="G$1" pin="1"/>
-<wire x1="109.22" y1="96.52" x2="93.98" y2="96.52" width="0.1524" layer="91"/>
-<wire x1="93.98" y1="96.52" x2="93.98" y2="119.38" width="0.1524" layer="91"/>
-<wire x1="93.98" y1="119.38" x2="96.52" y2="119.38" width="0.1524" layer="91"/>
-<junction x="109.22" y="45.72"/>
 </segment>
 </net>

Commit message: Допиливание железа
Подтяжки TX на Vcc, забытый резистор на верхнем транзисторе в драйвере,
конденсаторы на питание МК, подписи элементов в разводке
Parts:
- added C2: 100nF, capacitor-wima:C2,5-3
- added R4: 2R2, resistor:R-EU_R1206
- added R5: 10K, resistor:R-EU_M1206
- R1: value (none) -> 10K
Connections:
- removed net +5V: U1.VCC
- new net N$12: Q1.C, R4.1
- net GND: now also C2.2
- net N$1: now also R5.2
- net VCC: now also C2.1, R4.2, R5.1, U1.VCC; no longer Q1.C
Changed lines of the file:
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@@
 <part name="GND1" library="supply1" deviceset="GND" device=""/>
 <part name="U1" library="Maxim_By_element14_Batch_1" deviceset="MAX485CSA+" device=""/>
-<part name="P+1" library="supply1" deviceset="+5V" device=""/>
 <part name="IC1" library="atmel" deviceset="MEGA8" device="-AI"/>
 <part name="ISP" library="con-molex" deviceset="5566-10" device=""/>
@@
 <part name="GND2" library="supply1" deviceset="GND" device=""/>
 <part name="P+4" library="supply1" deviceset="VCC" device=""/>
-<part name="R1" library="resistor" deviceset="R-EU_" device="M1206"/>
+<part name="R1" library="resistor" deviceset="R-EU_" device="M1206" value="10K"/>
 <part name="GND3" library="supply1" deviceset="GND" device=""/>
 <part name="R2" library="resistor" deviceset="R-EU_" device="R1206" value="22"/>
@@
 <part name="F1" library="fuse" deviceset="TE5" device=""/>
 <part name="LED" library="con-molex" deviceset="5566-10" device=""/>
+<part name="R4" library="resistor" deviceset="R-EU_" device="R1206" value="2R2"/>
+<part name="P+6" library="supply1" deviceset="VCC" device=""/>
+<part name="C2" library="capacitor-wima" deviceset="C" device="2,5-3" value="100nF"/>
+<part name="GND6" library="supply1" deviceset="GND" device=""/>
+<part name="P+1" library="supply1" deviceset="VCC" device=""/>
+<part name="P+7" library="supply1" deviceset="VCC" device=""/>
+<part name="R5" library="resistor" deviceset="R-EU_" device="M1206" value="10K"/>
 </parts>
 <sheets>
@@
 <instance part="GND1" gate="1" x="30.48" y="-7.62"/>
 <instance part="U1" gate="A" x="50.8" y="10.16"/>
-<instance part="P+1" gate="1" x="30.48" y="20.32"/>
 <instance part="IC1" gate="G$1" x="40.64" y="73.66"/>
 <instance part="ISP" gate="-1" x="121.92" y="66.04" smashed="yes">
@@
 <instance part="Q1" gate="1" x="114.3" y="127"/>
 <instance part="Q2" gate="G$1" x="114.3" y="111.76"/>
-<instance part="P+3" gate="VCC" x="116.84" y="137.16" smashed="yes">
-<attribute name="VALUE" x="114.3" y="134.62" size="1.778" layer="96" rot="R90"/>
+<instance part="P+3" gate="VCC" x="116.84" y="149.86" smashed="yes">
+<attribute name="VALUE" x="114.3" y="147.32" size="1.778" layer="96" rot="R90"/>
 </instance>
 <instance part="GND4" gate="1" x="116.84" y="101.6"/>
@@
 </instance>
 <instance part="LED" gate="-2" x="172.72" y="129.54"/>
+<instance part="R4" gate="G$1" x="116.84" y="139.7" rot="R90"/>
+<instance part="P+6" gate="VCC" x="0" y="96.52" smashed="yes">
+<attribute name="VALUE" x="-2.54" y="93.98" size="1.778" layer="96" rot="R90"/>
+</instance>
+<instance part="C2" gate="G$1" x="0" y="88.9"/>
+<instance part="GND6" gate="1" x="0" y="78.74"/>
+<instance part="P+1" gate="VCC" x="30.48" y="20.32" smashed="yes">
+<attribute name="VALUE" x="27.94" y="17.78" size="1.778" layer="96" rot="R90"/>
+</instance>
+<instance part="P+7" gate="VCC" x="10.16" y="22.86" smashed="yes">
+<attribute name="VALUE" x="7.62" y="20.32" size="1.778" layer="96" rot="R90"/>
+</instance>
+<instance part="R5" gate="G$1" x="10.16" y="12.7" rot="R270"/>
 </instances>
 <busses>
@@
 <pinref part="IC1" gate="G$1" pin="PD1(TXD)"/>
 <wire x1="66.04" y1="73.66" x2="88.9" y2="73.66" width="0.1524" layer="91"/>
+<pinref part="R5" gate="G$1" pin="2"/>
+<wire x1="17.78" y1="2.54" x2="10.16" y2="2.54" width="0.1524" layer="91"/>
+<wire x1="10.16" y1="2.54" x2="10.16" y2="7.62" width="0.1524" layer="91"/>
+<junction x="17.78" y="2.54"/>
 </segment>
 </net>
@@
 <segment>
 <pinref part="P+3" gate="VCC" pin="VCC"/>
-<pinref part="Q1" gate="1" pin="C"/>
-<wire x1="116.84" y1="134.62" x2="116.84" y2="132.08" width="0.1524" layer="91"/>
+<pinref part="R4" gate="G$1" pin="2"/>
+<wire x1="116.84" y1="147.32" x2="116.84" y2="144.78" width="0.1524" layer="91"/>
+</segment>
+<segment>
+<pinref part="P+6" gate="VCC" pin="VCC"/>
+<pinref part="C2" gate="G$1" pin="1"/>
+<wire x1="0" y1="93.98" x2="0" y2="91.44" width="0.1524" layer="91"/>
+</segment>
+<segment>
+<wire x1="33.02" y1="15.24" x2="30.48" y2="15.24" width="0.1524" layer="91"/>
+<pinref part="U1" gate="A" pin="VCC"/>
+<wire x1="30.48" y1="15.24" x2="30.48" y2="17.78" width="0.1524" layer="91"/>
+<pinref part="P+1" gate="VCC" pin="VCC"/>
+</segment>
+<segment>
+<pinref part="P+7" gate="VCC" pin="VCC"/>
+<pinref part="R5" gate="G$1" pin="1"/>
+<wire x1="10.16" y1="20.32" x2="10.16" y2="17.78" width="0.1524" layer="91"/>
 </segment>
 </net>
@@
 <wire x1="147.32" y1="116.84" x2="147.32" y2="114.3" width="0.1524" layer="91"/>
 </segment>
-</net>
-<net name="+5V" class="0">
-<segment>
-<wire x1="33.02" y1="15.24" x2="30.48" y2="15.24" width="0.1524" layer="91"/>
-<pinref part="U1" gate="A" pin="VCC"/>
-<pinref part="P+1" gate="1" pin="+5V"/>
-<wire x1="30.48" y1="15.24" x2="30.48" y2="17.78" width="0.1524" layer="91"/>
+<segment>
+<pinref part="C2" gate="G$1" pin="2"/>
+<pinref part="GND6" gate="1" pin="GND"/>
+<wire x1="0" y1="83.82" x2="0" y2="81.28" width="0.1524" layer="91"/>
 </segment>
 </net>
@@
 </segment>
 </net>
+<net name="N$12" class="0">
+<segment>
+<pinref part="R4" gate="G$1" pin="1"/>
+<pinref part="Q1" gate="1" pin="C"/>
+<wire x1="116.84" y1="134.62" x2="116.84" y2="132.08" width="0.1524" layer="91"/>
+</segment>
+</net>
