File: wrk/led driver.sch (EAGLE design)
At the start: 15 parts, among them IC1 MEGA8-AI, Q1 BCP56, Q2 BCP53, Q3 IRF540, U1 MAX485CSA+

Commit message: бутерброд - основная плата и драйвер
Parts:
- removed C2: 100nF, capacitor-wima:C2,5-3
- removed IC1: MEGA8-AI, atmel:MEGA8-AI
- removed ISP: 5566-10, con-molex:5566-10
- removed R1, R5: 10K, resistor:R-EU_M1206
- removed U1: MAX485CSA+, Maxim_By_element14_Batch_1:MAX485CSA+
- added PIN15: 5566-10, con-molex:5566-10
Connections:
- removed net N$1: IC1.PD1(TXD), R5.2, U1.DI
- removed net N$11: IC1.PC6(/RESET), ISP-5.S, R1.2
- removed net N$2: IC1.PD0(RXD), U1.RO
- removed net N$3: IC1.PD2(INT0), U1.DE, U1.~RE
- removed net N$4: IC1.PB5(SCK), ISP-7.S
- removed net N$7: IC1.PB4(MISO), ISP-9.S
- net GND: no longer C2.2, IC1.GND, IC1.GND@1, IC1.GND@2, ISP-10.S, ISP-4.S, ISP-6.S, ISP-8.S, U1.GND
- net N$6: now also PIN15-1.S; no longer IC1.PB3(MOSI/OC2), ISP-1.S
- net VCC: no longer C2.1, IC1.AREF, IC1.AVCC, IC1.VCC@1, IC1.VCC@2, ISP-2.S, R1.1, R5.1, U1.VCC
Other:
- moved on the sheet: C1, F1, LED-1, LED-2, Q1, Q2, Q3, R2, R3, R4
